Commit message: Improve compatibility with Ubuntu 20.04

File: src/mybot_description/urdf/macros.xacro (robot description, xacro)
@@ -1,15 +1,15 @@
 <?xml version="1.0"?>
-<robot>
-     <macro name="cylinder_inertia" params="m r h">
+<robot xmlns:xacro="http://www.ros.org/wiki/xacro">
+     <xacro:macro name="cylinder_inertia" params="m r h">
         <inertia  ixx="${m*(3*r*r+h*h)/12}" ixy = "0" ixz = "0"
                   iyy="${m*(3*r*r+h*h)/12}" iyz = "0"
                   izz="${m*r*r/2}" />
-      </macro>
-      <macro name="box_inertia" params="m x y z">
+      </xacro:macro>
+      <xacro:macro name="box_inertia" params="m x y z">
         <inertia  ixx="${m*(y*y+z*z)/12}" ixy = "0" ixz = "0"
                   iyy="${m*(x*x+z*z)/12}" iyz = "0"
                   izz="${m*(x*x+y*y)/12}" />
-      </macro>
-    <macro name="wheel" params="lr fb tX tY">
+      </xacro:macro>
+    <xacro:macro name="wheel" params="lr fb tX tY">
       <link name="${lr}_${fb}_wheel">
         <collision>
@@ -29,5 +29,5 @@
           <origin xyz="0 0 0" rpy="0 ${PI/2} ${PI/2}" />
           <mass value="${wheelMass}"/>
-          <cylinder_inertia m="${wheelMass}" r="${wheelRadius}" h="${wheelWidth}"/>
+          <xacro:cylinder_inertia m="${wheelMass}" r="${wheelRadius}" h="${wheelWidth}"/>
         </inertial>
       </link>
@@ -59,6 +59,6 @@
         </actuator>
       </transmission>
-    </macro>
-    <macro name="wheel_trailer" params="lr fb tX tY dist">
+    </xacro:macro>
+    <xacro:macro name="wheel_trailer" params="lr fb tX tY dist">
       <link name="${lr}_${fb}_trailer_wheel">
         <collision>
@@ -98,4 +98,4 @@
         <dynamics damping="0.0" friction="0.0"/>
       </joint>
-    </macro>
+    </xacro:macro>
 </robot>

File: src/mybot_description/urdf/mybot.xacro (robot description, xacro)
@@ -58,11 +58,11 @@
       <origin xyz="0 0 0.2275" rpy="0 0 0"/>
       <mass value="${chassisMass}"/>
-      <box_inertia m="${chassisMass}" x="${chassisLength}" y="${chassisWidth}" z="${chassisHeight}"/>
+      <xacro:box_inertia m="${chassisMass}" x="${chassisLength}" y="${chassisWidth}" z="${chassisHeight}"/>
     </inertial>
   </link>
-  <wheel lr="left" fb="front" tX="0.25" tY="-0.3175"/>
-  <wheel lr="left" fb="back" tX="-0.25" tY="-0.3175"/>
-  <wheel lr="right" fb="front" tX="0.25" tY="0.3175"/>
-  <wheel lr="right" fb="back" tX="-0.25" tY="0.3175"/>
+  <xacro:wheel lr="left" fb="front" tX="0.25" tY="-0.3175"/>
+  <xacro:wheel lr="left" fb="back" tX="-0.25" tY="-0.3175"/>
+  <xacro:wheel lr="right" fb="front" tX="0.25" tY="0.3175"/>
+  <xacro:wheel lr="right" fb="back" tX="-0.25" tY="0.3175"/>
   <joint name="camera_joint" type="fixed">
     <origin xyz="${-cameraSize/2+chassisLength/2} 0 ${0.88-cameraSize/2}" rpy="0 ${PI/4} 0"/>
@@ -87,5 +87,5 @@
       <mass value="${cameraMass}" />
       <origin xyz="0 0 0" rpy="0 0 0"/>
-      <box_inertia m="${cameraMass}" x="${cameraSize}" y="${cameraSize}" z="${cameraSize}" />
+      <xacro:box_inertia m="${cameraMass}" x="${cameraSize}" y="${cameraSize}" z="${cameraSize}" />
     </inertial>
   </link>
@@ -112,5 +112,5 @@
       <mass value="${cameraMass}" />
       <origin xyz="0 0 0" rpy="0 0 0"/>
-      <box_inertia m="${cameraMass}" x="${cameraSize}" y="${cameraSize}" z="${cameraSize}" />
+      <xacro:box_inertia m="${cameraMass}" x="${cameraSize}" y="${cameraSize}" z="${cameraSize}" />
     </inertial>
   </link>
@@ -137,5 +137,5 @@
       <mass value="${cameraMass}" />
       <origin xyz="0 0 0" rpy="0 0 0"/>
-      <box_inertia m="${cameraMass}" x="${cameraSize}" y="${cameraSize}" z="${cameraSize/4}" />
+      <xacro:box_inertia m="${cameraMass}" x="${cameraSize}" y="${cameraSize}" z="${cameraSize/4}" />
     </inertial>
   </link>
